Commit message: Added RPLidar launch file, other fixes

File: ROS/warebot/warebot_lidar/urdf/model.urdf (robot description, URDF)
Before this commit: robot warebot, 3 links, 2 joints
Links:
- added link lidar_generic, mass 0.5
Joints:
- added joint lidar_base: type fixed, parent chassis, child lidar_generic, origin xyz=0.15 0 0.09 rpy=0 0 0, axis 0 0 1

Commit message: Added odometry via lidar, slam via gmapping for lidar setup

File: ROS/warebot/warebot_lidar/urdf/model.urdf (robot description, URDF)
Before this commit: robot warebot, 4 links, 3 joints
Links:
- removed link lidar_generic
- added link laser, mass 0.5
Joints:
- joint lidar_base: child lidar_generic -> laser

Commit message: Removed wheel joints, use laser filter for lidar, added laser scan matching

File: ROS/warebot/warebot_lidar/urdf/model.urdf (robot description, URDF)
Before this commit: robot warebot, 4 links, 3 joints
Links:
- removed link wheel_left
- removed link wheel_right
Joints:
- removed joint wheel_left_hinge
- removed joint wheel_right_hinge
