Commit message: tweaked pathfinding, added a world, etc

File: ROS/warebot/warebot_description/urdf/model.urdf (robot description, URDF)
Before this commit: robot warebot, 4 links, 3 joints
Joints:
- joint wheel_left_hinge: limit effort=20 velocity=50 -> effort=90 velocity=20
- joint wheel_right_hinge: limit effort=20 velocity=50 -> effort=90 velocity=20

Commit message: Final

File: ROS/warebot/warebot_description/urdf/model.urdf (robot description, URDF)
Before this commit: robot warebot, 4 links, 3 joints
Links:
- removed link lidar_generic
- added link laser, mass 0.5
Joints:
- joint lidar_base: child lidar_generic -> laser

File: ROS/warebot/warebot_description/urdf/real.urdf (robot description, URDF)
Before this commit: robot warebot, 2 links, 1 joints
Joints:
- joint lidar_base: origin xyz=0.15 0 0.12 rpy=0 0 -3.14158 -> xyz=0.10 0 0.12 rpy=0 0 0
